Commit message: Add crawler_robot_ros and LICENSE files

File: src/centaur/urdf/centaur.urdf (robot description, URDF)
Before this commit: robot centaur, 49 links, 48 joints
Links:
- link head_cam_link: geometry collision mesh filename=package://centaur/meshes/centaur/asus_camera_simple.dae; visual mesh filename=package://centaur/meshes/centaur/asus_camera_simple.dae
- link head_link: geometry collision mesh filename=package://centaur/meshes/centaur/multisensor_head_collision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 scale=0.001 0.001 0.001; visual mesh filename=package://centaur/meshes/centaur/multisensor_head.stl scale=0.001 0.001 0.001
- link head_link_hokuyo_laser_frame: geometry collision box size=0.058 0.058 0.087; visual mesh filename=package://centaur/meshes/centaur/hokuyo_utm_30lx.dae
- link infrared_frame: geometry collision mesh filename=package://centaur/meshes/centaur/thermaleye_camera_hector_v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; visual mesh filename=package://centaur/meshes/centaur/thermaleye_camera_hector_v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
- link l_arm_elbow: geometry collision box size=0.06 0.13 0.08; visual mesh filename=package://centaur/meshes/centaur/elbow_left_mod.stl scale=0.001 0.001 0.001
- link l_arm_shoulder_pitch: geometry collision box size=0.16 0.085 0.06; visual mesh filename=package://centaur/meshes/centaur/shoulder_pitch_left.stl scale=0.001 0.001 0.001
- link l_arm_shoulder_roll: geometry collision box size=0.16 0.06 0.06; visual mesh filename=package://centaur/meshes/centaur/shoulder_roll_left.stl scale=0.001 0.001 0.001
- link l_arm_shoulder_yaw: geometry collision box size=0.06 0.13 0.06; collision box size=0.08 0.08 0.204
- link l_arm_wrist_roll: geometry collision box size=0.06 0.06 0.10; collision box size=0.1 0.06 0.06
- link l_arm_wrist_yaw: geometry collision box size=0.06 0.06 0.10; collision box size=0.1 0.06 0.06
- link l_f0_link_0: geometry collision cylinder length=0.02 radius=0.014; collision cylinder length=0.02 radius=0.017
- link l_f1_link_0: geometry collision cylinder length=0.02 radius=0.014; collision cylinder length=0.02 radius=0.017
- link l_palm: geometry collision mesh filename=package://centaur/meshes/centaur/l_palm.stl; visual mesh filename=package://centaur/meshes/centaur/l_palm.stl
- link laser1_frame: geometry collision box size=0.058 0.058 0.087; visual mesh filename=package://centaur/meshes/centaur/hokuyo_utm_30lx.dae
- link neck_link: geometry collision box size=0.045 0.045 0.15; visual mesh filename=package://centaur/meshes/centaur/neck.stl scale=0.001 0.001 0.001
- link openni_link: geometry collision mesh filename=package://centaur/meshes/centaur/asus_camera_simple.dae; visual mesh filename=package://centaur/meshes/centaur/asus_camera_simple.dae
- link pelvis: geometry collision box size=0.23 0.23 0.24; visual mesh filename=package://centaur/meshes/centaur/pelvis.stl scale=0.001 0.001 0.001
- link r_arm_elbow: geometry collision box size=0.06 0.13 0.08; visual mesh filename=package://centaur/meshes/centaur/elbow_left_mod.stl scale=0.001 0.001 0.001
- link r_arm_shoulder_pitch: geometry collision box size=0.16 0.085 0.06; visual mesh filename=package://centaur/meshes/centaur/shoulder_pitch_left.stl scale=0.001 -0.001 0.001
- link r_arm_shoulder_roll: geometry collision box size=0.16 0.06 0.06; visual mesh filename=package://centaur/meshes/centaur/shoulder_roll_left.stl scale=0.001 0.001 0.001
- link r_arm_shoulder_yaw: geometry collision box size=0.06 0.13 0.06; collision box size=0.08 0.08 0.204
- link r_arm_wrist_roll: geometry collision box size=0.06 0.06 0.10; collision box size=0.1 0.06 0.06
- link r_arm_wrist_yaw: geometry collision box size=0.06 0.06 0.10; collision box size=0.1 0.06 0.06
- link r_f0_link_0: geometry collision cylinder length=0.02 radius=0.014; collision cylinder length=0.02 radius=0.017
- link r_f1_link_0: geometry collision cylinder length=0.02 radius=0.014; collision cylinder length=0.02 radius=0.017
- link r_palm: geometry collision mesh filename=package://centaur/meshes/centaur/r_palm.stl; visual mesh filename=package://centaur/meshes/centaur/r_palm.stl
- link utorso: geometry collision box size=0.24 0.31 0.24; collision cylinder length=0.23 radius=0.04
- link waist: geometry collision box size=0.03 0.08 0.03; visual mesh filename=package://centaur/meshes/centaur/waist.stl scale=0.001 0.001 0.001
