Commit message: fix quadrotor.urdf

File: src/quadrotor/urdf/quadrotor.urdf (robot description, URDF)
Before this commit: robot quadrotor, 5 links, 4 joints
Links:
- link base_link: geometry collision mesh filename=package://quadrotor/meshes/quadrotor/quadrotor_base.stl; visual mesh filename=package://quadrotor/meshes/quadrotor/quadrotor_base.dae
- link sonar_link: geometry collision box size=0.01 0.01 0.01; visual mesh filename=package://quadrotor/meshes/quadrotor/max_sonar_ez4.dae
