Commit message: fix urdf

File: src/crawler_robot_ros/urdf/crawler_robot.urdf (robot description, URDF)
Before this commit: robot crawler_robot, 31 links, 30 joints
Links:
- removed link crawler_robot__camera_ros_link
- removed link crawler_robot__chassis
- removed link crawler_robot__hokuyo_ros_link
- removed link crawler_robot__left_center_wheel_1
- removed link crawler_robot__left_center_wheel_2
- removed link crawler_robot__left_front_arm
- removed link crawler_robot__left_front_arm_wheel_1
- removed link crawler_robot__left_front_arm_wheel_2
- removed link crawler_robot__left_front_arm_wheel_3
- removed link crawler_robot__left_front_wheel
- removed link crawler_robot__left_rear_arm
- removed link crawler_robot__left_rear_arm_wheel_1
- removed link crawler_robot__left_rear_arm_wheel_2
- removed link crawler_robot__left_rear_arm_wheel_3
- removed link crawler_robot__left_rear_wheel
- removed link crawler_robot__left_sub_wheel_2
- removed link crawler_robot__left_sub_wheel_3
- removed link crawler_robot__right_center_wheel_1
- removed link crawler_robot__right_center_wheel_2
- removed link crawler_robot__right_front_arm
- removed link crawler_robot__right_front_arm_wheel_1
- removed link crawler_robot__right_front_arm_wheel_2
- removed link crawler_robot__right_front_arm_wheel_3
- removed link crawler_robot__right_front_wheel
- removed link crawler_robot__right_rear_arm
- removed link crawler_robot__right_rear_arm_wheel_1
- removed link crawler_robot__right_rear_arm_wheel_2
- removed link crawler_robot__right_rear_arm_wheel_3
- removed link crawler_robot__right_rear_wheel
- removed link crawler_robot__right_sub_wheel_2
- removed link crawler_robot__right_sub_wheel_3
- added link base_link, mass 20; collision box size=.1 .32 .06; visual box size=.1 .32 .06
- added link camera_link, mass 0.1; collision box size=0.08 0.1 0.1; collision cylinder length=0.02 radius=0.03
- added link hokuyo_link, mass 0.1; collision box size=0.05 0.05 0.041; collision cylinder length=0.029 radius=0.021
- added link left_center_wheel_1, mass 1.0; collision cylinder length=.05 radius=.05
- added link left_center_wheel_2, mass 1.0; collision cylinder length=.05 radius=.05
- added link left_center_wheel_3, mass 1.0; collision cylinder length=.05 radius=.05
- added link left_front_arm, mass 1.0; visual box size=.002 .16 .05; visual mesh filename=package://crawler_robot_ros/meshes/crawler_robot_ros/arm_cr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 scale=1.0 1.0 1.0
- added link left_front_arm_wheel_1, mass 1.0; collision cylinder length=.03 radius=.05; visual cylinder length=.03 radius=.05
- added link left_front_arm_wheel_2, mass 1.0; collision cylinder length=.03 radius=.05; visual cylinder length=.03 radius=.05
- added link left_front_arm_wheel_3, mass 1.0; collision cylinder length=.03 radius=.05
- added link left_front_wheel, mass 1.0; collision cylinder length=.1 radius=.05; visual cylinder length=.1 radius=.05
- added link left_rear_arm, mass 1.0; visual box size=.002 .16 .05; visual mesh filename=package://crawler_robot_ros/meshes/crawler_robot_ros/arm_cr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 scale=1.0 1.0 1.0
- added link left_rear_arm_wheel_1, mass 1.0; collision cylinder length=.03 radius=.05; visual cylinder length=.03 radius=.05
- added link left_rear_arm_wheel_2, mass 1.0; collision cylinder length=.03 radius=.05; visual cylinder length=.03 radius=.05
- added link left_rear_arm_wheel_3, mass 1.0; collision cylinder length=.03 radius=.05
- added link left_rear_wheel, mass 1.0; collision cylinder length=.1 radius=.05; visual cylinder length=.1 radius=.05
- added link left_sub_wheel_2, mass 1.0; collision cylinder length=.1 radius=.05
- added link left_sub_wheel_3, mass 1.0; collision cylinder length=.1 radius=.05
- added link right_center_wheel_1, mass 1.0; collision cylinder length=.05 radius=.05
- added link right_center_wheel_2, mass 1.0; collision cylinder length=.05 radius=.05
- added link right_center_wheel_3, mass 1.0; collision cylinder length=.05 radius=.05
- added link right_front_arm, mass 1.0; visual box size=.002 .16 .05; visual mesh filename=package://crawler_robot_ros/meshes/crawler_robot_ros/arm_cr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 scale=1.0 1.0 1.0
- added link right_front_arm_wheel_1, mass 1.0; collision cylinder length=.03 radius=.05; visual cylinder length=.03 radius=.05
- added link right_front_arm_wheel_2, mass 1.0; collision cylinder length=.03 radius=.05; visual cylinder length=.03 radius=.05
- added link right_front_arm_wheel_3, mass 1.0; collision cylinder length=.03 radius=.05
- added link right_front_wheel, mass 1.0; collision cylinder length=.1 radius=.05; visual cylinder length=.1 radius=.05
- added link right_rear_arm, mass 1.0; visual box size=.002 .16 .05; visual mesh filename=package://crawler_robot_ros/meshes/crawler_robot_ros/arm_cr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 scale=1.0 1.0 1.0
- added link right_rear_arm_wheel_1, mass 1.0; collision cylinder length=.03 radius=.05; visual cylinder length=.03 radius=.05
- added link right_rear_arm_wheel_2, mass 1.0; collision cylinder length=.03 radius=.05; visual cylinder length=.03 radius=.05
- added link right_rear_arm_wheel_3, mass 1.0; collision cylinder length=.03 radius=.05
- added link right_rear_wheel, mass 1.0; collision cylinder length=.1 radius=.05; visual cylinder length=.1 radius=.05
- added link right_sub_wheel_2, mass 1.0; collision cylinder length=.1 radius=.05
- added link right_sub_wheel_3, mass 1.0; collision cylinder length=.1 radius=.05
Joints:
- removed joint crawler_robot__camera_joint
- removed joint crawler_robot__hokuyo_joint
- removed joint crawler_robot__left_center1
- removed joint crawler_robot__left_center2
- removed joint crawler_robot__left_front
- removed joint crawler_robot__left_front_arm
- removed joint crawler_robot__left_front_arm_wheel_1
- removed joint crawler_robot__left_front_arm_wheel_2
- removed joint crawler_robot__left_front_arm_wheel_3
- removed joint crawler_robot__left_rear
- removed joint crawler_robot__left_rear_arm
- removed joint crawler_robot__left_rear_arm_wheel_1
- removed joint crawler_robot__left_rear_arm_wheel_2
- removed joint crawler_robot__left_rear_arm_wheel_3
- removed joint crawler_robot__left_sub2
- removed joint crawler_robot__left_sub3
- removed joint crawler_robot__right_center1
- removed joint crawler_robot__right_center2
- removed joint crawler_robot__right_front
- removed joint crawler_robot__right_front_arm
- removed joint crawler_robot__right_front_arm_wheel_1
- removed joint crawler_robot__right_front_arm_wheel_2
- removed joint crawler_robot__right_front_arm_wheel_3
- removed joint crawler_robot__right_rear
- removed joint crawler_robot__right_rear_arm
- removed joint crawler_robot__right_rear_arm_wheel_1
- removed joint crawler_robot__right_rear_arm_wheel_2
- removed joint crawler_robot__right_rear_arm_wheel_3
- removed joint crawler_robot__right_sub2
- removed joint crawler_robot__right_sub3
- added joint camera_joint: type fixed, parent base_link, child camera_link, origin xyz=0    0    0.22 rpy=0    0   -1.57, axis 0  0  1, limit lower=0.0 upper=0.0 effort=0.0 velocity=0.0
- added joint hokuyo_joint: type fixed, parent base_link, child hokuyo_link, origin xyz=0     0     0.135 rpy=0    0   -1.57, axis 0  0  1, limit lower=0.0 upper=0.0 effort=0.0 velocity=0.0
- added joint left_center1: type fixed, parent base_link, child left_center_wheel_1, origin xyz=0.05  0.05  0.05 rpy=3.14159  1.57079  3.14159, axis 0  0  1, limit lower=0 upper=0 effort=0 velocity=0
- added joint left_center2: type fixed, parent base_link, child left_center_wheel_2, origin xyz=0.05   0     0.049 rpy=3.14159  1.57079  3.14159, axis 0  0  1, limit lower=0 upper=0 effort=0 velocity=0
- added joint left_center3: type fixed, parent base_link, child left_center_wheel_3, origin xyz=0.05 -0.05  0.05 rpy=3.14159  1.57079  3.14159, axis 0  0  1, limit lower=0 upper=0 effort=0 velocity=0
- added joint left_front: type fixed, parent base_link, child left_front_wheel, origin xyz=0.05 -0.15  0.05 rpy=3.14159  1.57079  3.14159, axis 0  0  1, limit lower=0 upper=0 effort=0 velocity=0
- added joint left_front_arm_joint: type revolute, parent base_link, child left_front_arm, origin xyz=0.151 -0.15   0.051 rpy=0  0  0, axis 1  0  0, limit lower=-3.14 upper=3.14 effort=0.0 velocity=1.0
- added joint left_front_arm_wheel_1: type fixed, parent left_front_arm, child left_front_arm_wheel_1, origin xyz=0     0    -0.001 rpy=3.14159  1.57079  3.14159, axis 0  0  1, limit lower=0 upper=0 effort=0 velocity=0
- added joint left_front_arm_wheel_2: type fixed, parent left_front_arm, child left_front_arm_wheel_2, origin xyz=0    -0.15  -0.001 rpy=3.14159  1.57079  3.14159, axis 0  0  1, limit lower=0 upper=0 effort=0 velocity=0
- added joint left_front_arm_wheel_3: type fixed, parent left_front_arm, child left_front_arm_wheel_3, origin xyz=0    -0.075 -0.001 rpy=3.14159  1.57079  3.14159, axis 0  0  1, limit lower=0 upper=0 effort=0 velocity=0
- added joint left_rear: type fixed, parent base_link, child left_rear_wheel, origin xyz=0.05  0.15  0.05 rpy=3.14159  1.57079  3.14159, axis 0  0  1, limit lower=0 upper=0 effort=0 velocity=0
- added joint left_rear_arm_joint: type revolute, parent base_link, child left_rear_arm, origin xyz=0.151  0.15   0.051 rpy=0  0  0, axis 1  0  0, limit lower=-3.14 upper=3.14 effort=0.0 velocity=1.0
- added joint left_rear_arm_wheel_1: type fixed, parent left_rear_arm, child left_rear_arm_wheel_1, origin xyz=0     0    -0.001 rpy=3.14159  1.57079  3.14159, axis 0  0  1, limit lower=0 upper=0 effort=0 velocity=0
- added joint left_rear_arm_wheel_2: type fixed, parent left_rear_arm, child left_rear_arm_wheel_2, origin xyz=0     0.15  -0.001 rpy=3.14159  1.57079  3.14159, axis 0  0  1, limit lower=0 upper=0 effort=0 velocity=0
- added joint left_rear_arm_wheel_3: type fixed, parent left_rear_arm, child left_rear_arm_wheel_3, origin xyz=0     0.075 -0.001 rpy=3.14159  1.57079  3.14159, axis 0  0  1, limit lower=0 upper=0 effort=0 velocity=0
- added joint left_sub2: type fixed, parent base_link, child left_sub_wheel_2, origin xyz=0.05  0.1   0.05 rpy=3.14159  1.57079  3.14159, axis 0  0  1, limit lower=0 upper=0 effort=0 velocity=0
- added joint left_sub3: type fixed, parent base_link, child left_sub_wheel_3, origin xyz=0.05 -0.1   0.05 rpy=3.14159  1.57079  3.14159, axis 0  0  1, limit lower=0 upper=0 effort=0 velocity=0
- added joint right_center1: type fixed, parent base_link, child right_center_wheel_1, origin xyz=-0.05  0.05  0.05 rpy=3.14159  1.57079  3.14159, axis 0  0  1, limit lower=0 upper=0 effort=0 velocity=0
- added joint right_center2: type fixed, parent base_link, child right_center_wheel_2, origin xyz=-0.05   0     0.049 rpy=3.14159  1.57079  3.14159, axis 0  0  1, limit lower=0 upper=0 effort=0 velocity=0
- added joint right_center3: type fixed, parent base_link, child right_center_wheel_3, origin xyz=-0.05 -0.05  0.05 rpy=3.14159  1.57079  3.14159, axis 0  0  1, limit lower=0 upper=0 effort=0 velocity=0
- added joint right_front: type fixed, parent base_link, child right_front_wheel, origin xyz=-0.05 -0.15  0.05 rpy=3.14159  1.57079  3.14159, axis 0  0  1, limit lower=0 upper=0 effort=0 velocity=0
- added joint right_front_arm_joint: type revolute, parent base_link, child right_front_arm, origin xyz=-0.151 -0.15   0.049 rpy=0  0  0, axis 1  0  0, limit lower=-3.14 upper=3.14 effort=0.0 velocity=1.0
- added joint right_front_arm_wheel_1: type fixed, parent right_front_arm, child right_front_arm_wheel_1, origin xyz=0     0     0.001 rpy=3.14159  1.57079  3.14159, axis 0  0  1, limit lower=0 upper=0 effort=0 velocity=0
- added joint right_front_arm_wheel_2: type fixed, parent right_front_arm, child right_front_arm_wheel_2, origin xyz=0    -0.15   0.001 rpy=3.14159  1.57079  3.14159, axis 0  0  1, limit lower=0 upper=0 effort=0 velocity=0
- added joint right_front_arm_wheel_3: type fixed, parent right_front_arm, child right_front_arm_wheel_3, origin xyz=0    -0.075  0.001 rpy=3.14159  1.57079  3.14159, axis 0  0  1, limit lower=0 upper=0 effort=0 velocity=0
- added joint right_rear: type fixed, parent base_link, child right_rear_wheel, origin xyz=-0.05  0.15  0.05 rpy=3.14159  1.57079  3.14159, axis 0  0  1, limit lower=0 upper=0 effort=0 velocity=0
- added joint right_rear_arm_joint: type revolute, parent base_link, child right_rear_arm, origin xyz=-0.151  0.15   0.049 rpy=0  0  0, axis 1  0  0, limit lower=-3.14 upper=3.14 effort=0.0 velocity=1.0
- added joint right_rear_arm_wheel_1: type fixed, parent right_rear_arm, child right_rear_arm_wheel_1, origin xyz=0     0     0.001 rpy=3.14159  1.57079  3.14159, axis 0  0  1, limit lower=0 upper=0 effort=0 velocity=0
- added joint right_rear_arm_wheel_2: type fixed, parent right_rear_arm, child right_rear_arm_wheel_2, origin xyz=0     0.15   0.001 rpy=3.14159  1.57079  3.14159, axis 0  0  1, limit lower=0 upper=0 effort=0 velocity=0
- added joint right_rear_arm_wheel_3: type fixed, parent right_rear_arm, child right_rear_arm_wheel_3, origin xyz=0     0.075  0.001 rpy=3.14159  1.57079  3.14159, axis 0  0  1, limit lower=0 upper=0 effort=0 velocity=0
- added joint right_sub2: type fixed, parent base_link, child right_sub_wheel_2, origin xyz=-0.15  0.1   0.05 rpy=3.14159  1.57079  3.14159, axis 0  0  1, limit lower=0 upper=0 effort=0 velocity=0
- added joint right_sub3: type fixed, parent base_link, child right_sub_wheel_3, origin xyz=-0.15 -0.1   0.05 rpy=3.14159  1.57079  3.14159, axis 0  0  1, limit lower=0 upper=0 effort=0 velocity=0
